File: ubmp_v1r1_panel.kicad_pcb (KiCad board)
At the start: 2 copper layers, 154.5 x 113.5 mm, 402 parts, among them J1 Conn_02x05_Counter_Clockwise, J2 USB_A, U1 STM32F103CBUx, U2 MIC5245-3.3, Y1 PRQC8.00CR1010V00L

Commit message: Testing more with panel
Other:
- outline, holes or cut-outs redrawn
