File: ubmp_v1r1.sch (KiCad schematic (older format))
At the start: 24 parts, among them J1 USB_A, J2 Conn_02x04_Top_Bottom, U1 STM32F103CBUx, U2 MIC5245-3.3, Y1 PRQC8.00CR1010V00L

Commit message: PCB layout done
Connections:
- net labels added: DM_P, DPU, DP_P, LED
Changed lines of the file:
@@
 EESchema Schematic File Version 4
+LIBS:ubmp_v1r1-cache
 EELAYER 26 0
 EELAYER END
@@
 $EndComp
 Connection ~ 10350 4550
+Text Label 8900 4300 0    50   ~ 0
+DP_P
+Text Label 8900 4200 0    50   ~ 0
+DM_P
+Text Label 8900 4100 0    50   ~ 0
+DPU
+Text Label 2350 2700 0    50   ~ 0
+LED
 $EndSCHEMATC

Commit message: Added OSHW + README
Changed lines of the file:
@@
 Text Label 2350 2700 0    50   ~ 0
 LED
+$Comp
+L Graphic:Logo_Open_Hardware_Small #LOGO1
+U 1 1 5A78D4B8
+P 850 7500
+F 0 "#LOGO1" H 850 7775 50  0001 C CNN
+F 1 "Logo_Open_Hardware_Small" H 850 7275 50  0001 C CNN
+F 2 "" H 850 7500 50  0001 C CNN
+F 3 "~" H 850 7500 50  0001 C CNN
+	1    850  7500
+	1    0    0    -1
+$EndComp
 $EndSCHEMATC

Commit message: Updated schematic for STLink V2 clone
Parts:
- removed J2: Conn_02x04_Top_Bottom, ubmp:2x5_2.54mm_side, symbol Connector_Generic:Conn_02x04_Top_Bottom
- removed R3: 470, Resistor_SMD:R_0402_1005Metric, symbol Device:R
- added D2: GREEN, Diode_SMD:D_0603_1608Metric, symbol Device:LED
- added J1: Conn_02x05_Counter_Clockwise, symbol Connector_Generic:Conn_02x05_Counter_Clockwise
- added R1, R12, R2, R5: 100, Resistor_SMD:R_0402_1005Metric, symbol Device:R
- added R8: 1.5k, Resistor_SMD:R_0402_1005Metric, symbol Device:R
- added TP1, TP2, TP3, TP4: Test_Point, TestPoint:TestPoint_Pad_D1.0mm, symbol Connector_Specialized:Test_Point
- R9: renamed from R11; value 100 -> 22
- renumbered J1 to J2, R12 to R10, R10 to R11, R8 to R13, R4 to R14, R5 to R15, R6 to R16, R7 to R3, R9 to R4, R1 to R6, R2 to R7
Connections:
- net labels added: BMP_SWCLK/TCK, BMP_SWDIO/TMS, BMP_TDI, BMP_TDO, LED_STLINK, LED_UART, SWCLK, SWDIO
- net labels removed: BMP_SWCLK, BMP_SWDIO, DPU, LED
- wire segments 79 -> 88
- no-connect marks 24 -> 21
Other:
- note added: "1.0"
- note added: "2018-02-16"
- note added: "MCO"
- note added: "RST resistor is 22 Ohm to support board with small (<1.5k) pullup on RST"
- note added: "STLink V2 identifier (PC13 = 0)"
- note added: "SWD Programming"
- note added: "µBMP"
- moved on the sheet: U2

Commit message: Updated board for STLink V2 clone, added schematic print, updated images, updated README
Parts:
- C5, C6: value 10u -> 4.7u
- J1: footprint (none) -> ubmp:2x5_2.54mm_side
Connections:
- net labels added: BMP_RSTo, BMP_RXo, BMP_SWCLK_TCK, BMP_SWCLK_TCKo, BMP_SWDIO_TMS, BMP_SWDIO_TMSo, BMP_SWOo, BMP_TDIo, BMP_TDOo, BMP_TXo, BOOT0, NRST, STM_ID
- net labels removed: BMP_SWCLK/TCK, BMP_SWDIO/TMS
- wire segments 88 -> 99
Other:
- note added: "Design available at: github.com/korken89/micro-bmp"
- note added: "Note that this board is designed to work with the \nSTLink V2 version of Black Magic Probe firmware."

Commit message: Fixed footprint associations in sch
Parts:
- C1, C2, C3, C4: footprint Capacitor_SMD:C_0402_1005Metric -> ubmp:C_0402_1005Metric_Rounded
- C5, C6: footprint Capacitor_SMD:C_0603_1608Metric -> ubmp:C_0603_1608Metric_Rounded
- D1, D2: footprint Diode_SMD:D_0603_1608Metric -> ubmp:D_0603_1608Metric_Rounded
- R1, R2: value 100 -> 470; footprint Resistor_SMD:R_0402_1005Metric -> ubmp:R_0402_1005Metric_Rounded
- R10, R11, R12, R13, R14, R15, R16, R3, R4, R5, R6, R7, R8, R9: footprint Resistor_SMD:R_0402_1005Metric -> ubmp:R_0402_1005Metric_Rounded
Changed lines of the file:
@@
 EESchema Schematic File Version 4
-LIBS:ubmp_v1r1-cache
 EELAYER 26 0
 EELAYER END
@@
 F 0 "C4" H 4592 1146 50  0000 L CNN
 F 1 "100n" H 4592 1055 50  0000 L CNN
-F 2 "Capacitor_SMD:C_0402_1005Metric" H 4500 1100 50  0001 C CNN
+F 2 "ubmp:C_0402_1005Metric_Rounded" H 4500 1100 50  0001 C CNN
 F 3 "~" H 4500 1100 50  0001 C CNN
 	1    4500 1100
@@
 F 0 "C3" H 4242 1146 50  0000 L CNN
 F 1 "100n" H 4242 1055 50  0000 L CNN
-F 2 "Capacitor_SMD:C_0402_1005Metric" H 4150 1100 50  0001 C CNN
+F 2 "ubmp:C_0402_1005Metric_Rounded" H 4150 1100 50  0001 C CNN
 F 3 "~" H 4150 1100 50  0001 C CNN
 	1    4150 1100
@@
 F 0 "C2" H 3892 1146 50  0000 L CNN
 F 1 "100n" H 3892 1055 50  0000 L CNN
-F 2 "Capacitor_SMD:C_0402_1005Metric" H 3800 1100 50  0001 C CNN
+F 2 "ubmp:C_0402_1005Metric_Rounded" H 3800 1100 50  0001 C CNN
 F 3 "~" H 3800 1100 50  0001 C CNN
 	1    3800 1100
@@
 F 0 "C1" H 3542 1146 50  0000 L CNN
 F 1 "100n" H 3542 1055 50  0000 L CNN
-F 2 "Capacitor_SMD:C_0402_1005Metric" H 3450 1100 50  0001 C CNN
+F 2 "ubmp:C_0402_1005Metric_Rounded" H 3450 1100 50  0001 C CNN
 F 3 "~" H 3450 1100 50  0001 C CNN
 	1    3450 1100
@@
 F 0 "C5" H 2742 7146 50  0000 L CNN
 F 1 "4.7u" H 2742 7055 50  0000 L CNN
-F 2 "Capacitor_SMD:C_0603_1608Metric" H 2650 7100 50  0001 C CNN
+F 2 "ubmp:C_0603_1608Metric_Rounded" H 2650 7100 50  0001 C CNN
 F 3 "~" H 2650 7100 50  0001 C CNN
 	1    2650 7100
@@
 F 0 "C6" H 3892 7146 50  0000 L CNN
 F 1 "4.7u" H 3892 7055 50  0000 L CNN
-F 2 "Capacitor_SMD:C_0603_1608Metric" H 3800 7100 50  0001 C CNN
+F 2 "ubmp:C_0603_1608Metric_Rounded" H 3800 7100 50  0001 C CNN
 F 3 "~" H 3800 7100 50  0001 C CNN
 	1    3800 7100
@@
 F 0 "R15" V 9750 4200 50  0000 C CNN
 F 1 "22" V 9850 4200 50  0000 C CNN
-F 2 "Resistor_SMD:R_0402_1005Metric" V 9780 4200 50  0001 C CNN
+F 2 "ubmp:R_0402_1005Metric_Rounded" V 9780 4200 50  0001 C CNN
 F 3 "~" H 9850 4200 50  0001 C CNN
 	1    9850 4200
@@
 F 0 "R16" V 9950 4300 50  0000 C CNN
 F 1 "22" V 9850 4300 50  0000 C CNN
-F 2 "Resistor_SMD:R_0402_1005Metric" V 9780 4300 50  0001 C CNN
+F 2 "ubmp:R_0402_1005Metric_Rounded" V 9780 4300 50  0001 C CNN
 F 3 "~" H 9850 4300 50  0001 C CNN
 	1    9850 4300
@@
 F 0 "D1" H 9800 1150 50  0000 C CNN
 F 1 "YELLOW" H 9800 900 50  0000 C CNN
-F 2 "Diode_SMD:D_0603_1608Metric" H 9800 1050 50  0001 C CNN
+F 2 "ubmp:D_0603_1608Metric_Rounded" H 9800 1050 50  0001 C CNN
 F 3 "~" H 9800 1050 50  0001 C CNN
 	1    9800 1050
@@
 F 0 "R7" V 2050 2000 50  0000 C CNN
 F 1 "1.5k" V 2150 2000 50  0000 C CNN
-F 2 "Resistor_SMD:R_0402_1005Metric" V 2080 2000 50  0001 C CNN
+F 2 "ubmp:R_0402_1005Metric_Rounded" V 2080 2000 50  0001 C CNN
 F 3 "~" H 2150 2000 50  0001 C CNN
 	1    2150 2000
@@
 F 0 "R6" V 2050 1800 50  0000 C CNN
 F 1 "1.5k" V 2150 1800 50  0000 C CNN
-F 2 "Resistor_SMD:R_0402_1005Metric" V 2080 1800 50  0001 C CNN
+F 2 "ubmp:R_0402_1005Metric_Rounded" V 2080 1800 50  0001 C CNN
 F 3 "~" H 2150 1800 50  0001 C CNN
 	1    2150 1800
@@
 F 0 "R3" V 1450 5100 50  0000 C CNN
 F 1 "100" V 1550 5100 50  0000 C CNN
-F 2 "Resistor_SMD:R_0402_1005Metric" V 1480 5100 50  0001 C CNN
+F 2 "ubmp:R_0402_1005Metric_Rounded" V 1480 5100 50  0001 C CNN
 F 3 "~" H 1550 5100 50  0001 C CNN
 	1    1550 5100
@@
 F 0 "R4" V 1700 5000 50  0000 C CNN
 F 1 "100" V 1800 5000 50  0000 C CNN
-F 2 "Resistor_SMD:R_0402_1005Metric" V 1730 5000 50  0001 C CNN
+F 2 "ubmp:R_0402_1005Metric_Rounded" V 1730 5000 50  0001 C CNN
 F 3 "~" H 1800 5000 50  0001 C CNN
 	1    1800 5000
@@
 F 0 "R9" V 1700 5200 50  0000 C CNN
 F 1 "22" V 1800 5200 50  0000 C CNN
-F 2 "Resistor_SMD:R_0402_1005Metric" V 1730 5200 50  0001 C CNN
+F 2 "ubmp:R_0402_1005Metric_Rounded" V 1730 5200 50  0001 C CNN
 F 3 "~" H 1800 5200 50  0001 C CNN
 	1    1800 5200
@@
 F 0 "R10" V 1450 5500 50  0000 C CNN
 F 1 "100" V 1550 5500 50  0000 C CNN
-F 2 "Resistor_SMD:R_0402_1005Metric" V 1480 5500 50  0001 C CNN
+F 2 "ubmp:R_0402_1005Metric_Rounded" V 1480 5500 50  0001 C CNN
 F 3 "~" H 1550 5500 50  0001 C CNN
 	1    1550 5500
@@
 F 0 "R11" V 1450 5700 50  0000 C CNN
 F 1 "100" V 1550 5700 50  0000 C CNN
-F 2 "Resistor_SMD:R_0402_1005Metric" V 1480 5700 50  0001 C CNN
+F 2 "ubmp:R_0402_1005Metric_Rounded" V 1480 5700 50  0001 C CNN
 F 3 "~" H 1550 5700 50  0001 C CNN
 	1    1550 5700
@@
 F 0 "R13" V 1700 5400 50  0000 C CNN
 F 1 "100" V 1800 5400 50  0000 C CNN
-F 2 "Resistor_SMD:R_0402_1005Metric" V 1730 5400 50  0001 C CNN
+F 2 "ubmp:R_0402_1005Metric_Rounded" V 1730 5400 50  0001 C CNN
 F 3 "~" H 1800 5400 50  0001 C CNN
 	1    1800 5400
@@
 F 0 "R5" V 1450 5300 50  0000 C CNN
 F 1 "100" V 1550 5300 50  0000 C CNN
-F 2 "Resistor_SMD:R_0402_1005Metric" V 1480 5300 50  0001 C CNN
+F 2 "ubmp:R_0402_1005Metric_Rounded" V 1480 5300 50  0001 C CNN
 F 3 "~" H 1550 5300 50  0001 C CNN
 	1    1550 5300
@@
 F 0 "R12" V 1700 5600 50  0000 C CNN
 F 1 "100" V 1800 5600 50  0000 C CNN
-F 2 "Resistor_SMD:R_0402_1005Metric" V 1730 5600 50  0001 C CNN
+F 2 "ubmp:R_0402_1005Metric_Rounded" V 1730 5600 50  0001 C CNN
 F 3 "~" H 1800 5600 50  0001 C CNN
 	1    1800 5600
@@
 P 10100 1050
 F 0 "R1" V 10000 1050 50  0000 C CNN
-F 1 "100" V 10100 1050 50  0000 C CNN
-F 2 "Resistor_SMD:R_0402_1005Metric" V 10030 1050 50  0001 C CNN
+F 1 "470" V 10100 1050 50  0000 C CNN
+F 2 "ubmp:R_0402_1005Metric_Rounded" V 10030 1050 50  0001 C CNN
 F 3 "~" H 10100 1050 50  0001 C CNN
 	1    10100 1050
@@
 F 0 "R8" V 2050 2700 50  0000 C CNN
 F 1 "1.5k" V 2150 2700 50  0000 C CNN
-F 2 "Resistor_SMD:R_0402_1005Metric" V 2080 2700 50  0001 C CNN
+F 2 "ubmp:R_0402_1005Metric_Rounded" V 2080 2700 50  0001 C CNN
 F 3 "~" H 2150 2700 50  0001 C CNN
 	1    2150 2700
@@
 F 0 "D2" H 9800 1550 50  0000 C CNN
 F 1 "GREEN" H 9800 1300 50  0000 C CNN
-F 2 "Diode_SMD:D_0603_1608Metric" H 9800 1450 50  0001 C CNN
+F 2 "ubmp:D_0603_1608Metric_Rounded" H 9800 1450 50  0001 C CNN
 F 3 "~" H 9800 1450 50  0001 C CNN
 	1    9800 1450
@@
 P 10100 1450
 F 0 "R2" V 10000 1450 50  0000 C CNN
-F 1 "100" V 10100 1450 50  0000 C CNN
-F 2 "Resistor_SMD:R_0402_1005Metric" V 10030 1450 50  0001 C CNN
+F 1 "470" V 10100 1450 50  0000 C CNN
+F 2 "ubmp:R_0402_1005Metric_Rounded" V 10030 1450 50  0001 C CNN
 F 3 "~" H 10100 1450 50  0001 C CNN
 	1    10100 1450
@@
 F 0 "R14" V 9950 3950 50  0000 C CNN
 F 1 "1.5k" V 10050 3950 50  0000 C CNN
-F 2 "Resistor_SMD:R_0402_1005Metric" V 9980 3950 50  0001 C CNN
+F 2 "ubmp:R_0402_1005Metric_Rounded" V 9980 3950 50  0001 C CNN
 F 3 "~" H 10050 3950 50  0001 C CNN
 	1    10050 3950

Commit message: Footprint fixes
Parts:
- U1: footprint Package_DFN_QFN:QFN-48-1EP_7x7mm_P0.5mm_EP5.15x5.15mm -> ubmp:QFN-48-1EP_7x7mm_P0.5mm_EP5.15x5.15mm
- U2: footprint Package_TO_SOT_SMD:SOT-23-5 -> ubmp:SOT-23-5_Rounded
Changed lines of the file:
@@
 F 0 "U1" H 2850 4950 50  0000 C CNN
 F 1 "STM32F103CBUx" H 8100 4950 50  0000 C CNN
-F 2 "Package_DFN_QFN:QFN-48-1EP_7x7mm_P0.5mm_EP5.15x5.15mm" H 8400 4875 50  0001 R TNN
+F 2 "ubmp:QFN-48-1EP_7x7mm_P0.5mm_EP5.15x5.15mm" H 8400 4875 50  0001 R TNN
 F 3 "http://www.st.com/st-web-ui/static/active/en/resource/technical/document/datasheet/CD00161566.pdf" H 5600 3200 50  0001 C CNN
 	1    5600 3200
@@
 F 0 "U2" H 3300 7392 50  0000 C CNN
 F 1 "MIC5245-3.3" H 3300 7301 50  0000 C CNN
-F 2 "Package_TO_SOT_SMD:SOT-23-5" H 3300 7375 50  0001 C CNN
+F 2 "ubmp:SOT-23-5_Rounded" H 3300 7375 50  0001 C CNN
 F 3 "http://ww1.microchip.com/downloads/en/devicedoc/mic5205.pdf" H 3300 7050 50  0001 C CNN
 	1    3300 7050

Commit message: Changed to USB connector, 1.6mm PCB was too thin
Parts:
- J2: footprint usbpcb:USBPCB -> usbpcb:USB_A_1001-011-01101
Changed lines of the file:
@@
 F 0 "J2" H 10706 4767 50  0000 C CNN
 F 1 "USB_A" H 10706 4676 50  0000 C CNN
-F 2 "usbpcb:USBPCB" H 10800 4250 50  0001 C CNN
+F 2 "usbpcb:USB_A_1001-011-01101" H 10800 4250 50  0001 C CNN
 F 3 "" H 10800 4250 50  0001 C CNN
 	1    10650 4300

Commit message: Now more compatible with STLink-v2
Changes:
* Fixed 0603 cap spacing
* Added fuse to 5V line
* Connected unused signals from STLink schematic
* Connected BOOT1 to GND
* Removed yellow LED
* Updated width of USB connector pads for easier soldering
Parts:
- removed D1: YELLOW, ubmp:D_0603_1608Metric_Rounded, symbol Device:LED
- added F1: MF-FSMF050X-2, ubmp:R_0603_1608Metric_Rounded, symbol Device:Polyfuse_Small
- added R17, R18, R19: 1.5k, ubmp:R_0402_1005Metric_Rounded, symbol Device:R
- R1: value 470 -> 100
Connections:
- net labels added: STLINK_AIN_1, STLINK_SWDIO_IN, STM_ID2
- net labels removed: LED_UART
- wire segments 99 -> 111
- no-connect marks 21 -> 17
Other:
- note added: "STLink compatibility"
Changed lines of the file:
@@
-$EndComp
-$Comp
-L Device:LED D1
-U 1 1 5A7A3B34
-P 9800 1050
-F 0 "D1" H 9800 1150 50  0000 C CNN
-F 1 "YELLOW" H 9800 900 50  0000 C CNN
-F 2 "ubmp:D_0603_1608Metric_Rounded" H 9800 1050 50  0001 C CNN
-F 3 "~" H 9800 1050 50  0001 C CNN
-	1    9800 1050
-	1    0    0    -1
-$EndComp
-$Comp
-L power:GND #PWR01
-U 1 1 5A7A3BB4
-P 9650 1050
-F 0 "#PWR01" H 9650 800 50  0001 C CNN
-F 1 "GND" V 9655 922 50  0000 R CNN
-F 2 "" H 9650 1050 50  0001 C CNN
-F 3 "" H 9650 1050 50  0001 C CNN
-	1    9650 1050
-	0    1    1    0
 $EndComp
 $Comp
@@
 L power:+5V #PWR08
 U 1 1 5A7B31E8
-P 3050 5850
-F 0 "#PWR08" H 3050 5700 50  0001 C CNN
-F 1 "+5V" V 3065 5978 50  0000 L CNN
-F 2 "" H 3050 5850 50  0001 C CNN
-F 3 "" H 3050 5850 50  0001 C CNN
-	1    3050 5850
-	0    -1   -1   0
+P 3000 5400
+F 0 "#PWR08" H 3000 5250 50  0001 C CNN
+F 1 "+5V" V 3015 5528 50  0000 L CNN
+F 2 "" H 3000 5400 50  0001 C CNN
+F 3 "" H 3000 5400 50  0001 C CNN
+	1    3000 5400
+	1    0    0    -1
 $EndComp
 $Comp
@@
 Text Label 8700 4200 0    50   ~ 0
 DM_P
-Text Label 10350 1050 0    50   ~ 0
-LED_UART
 $Comp
 L Graphic:Logo_Open_Hardware_Small #LOGO1
@@
 	1650 5600 1300 5600
 $Comp
-L Device:R R1
-U 1 1 5A7CDD33
-P 10100 1050
-F 0 "R1" V 10000 1050 50  0000 C CNN
-F 1 "470" V 10100 1050 50  0000 C CNN
-F 2 "ubmp:R_0402_1005Metric_Rounded" V 10030 1050 50  0001 C CNN
-F 3 "~" H 10100 1050 50  0001 C CNN
-	1    10100 1050
-	0    1    1    0
-$EndComp
-$Comp
 L Device:R R8
 U 1 1 5A7CDF1D
@@
 	2500 3100 2700 3100
 Wire Wire Line
-	2700 4500 2500 4500
+	2700 4500 2550 4500
 Wire Wire Line
 	8700 3300 8500 3300
@@
 NoConn ~ 2700 2900
 NoConn ~ 2700 3200
-NoConn ~ 2700 3300
 NoConn ~ 2700 3400
 NoConn ~ 2700 3500
@@
 NoConn ~ 2700 4100
 NoConn ~ 2700 4200
-NoConn ~ 2700 4300
-NoConn ~ 2700 4400
 NoConn ~ 2700 4600
-NoConn ~ 8500 3100
 NoConn ~ 8500 3200
 NoConn ~ 8500 3500
@@
 Text Notes 9100 5600 0    50   ~ 0
 SWD Programming
-Text Notes 8700 3900 0    67   ~ 0
+Text Notes 8700 3900 0    50   ~ 0
 MCO
-Wire Wire Line
-	10250 1050 10350 1050
-Text Label 2500 2850 2    50   ~ 0
-LED_UART
-Wire Wire Line
-	2500 2850 2550 2850
-Wire Wire Line
-	2550 2850 2550 2800
-Wire Wire Line
-	2550 2800 2700 2800
 Wire Wire Line
 	8500 4300 9700 4300
@@
 Wire Wire Line
 	3600 6950 3800 6950
-Text Label 2350 1800 0    67   ~ 0
+Text Label 2350 1800 0    50   ~ 0
 NRST
-Text Label 2350 2000 0    67   ~ 0
+Text Label 2350 2000 0    50   ~ 0
 BOOT0
 Wire Wire Line
@@
 Wire Wire Line
 	2300 2700 2700 2700
-Text Label 2350 2700 0    67   ~ 0
+Text Label 2350 2700 0    50   ~ 0
 STM_ID
 Text Label 2100 5100 0    50   ~ 0
@@
 Text Notes 7100 7050 0    79   ~ 0
 Design available at: github.com/korken89/micro-bmp
+$Comp
+L Device:Polyfuse_Small F1
+U 1 1 5AB80C43
+P 3000 5500
+F 0 "F1" H 2932 5454 50  0000 R CNN
+F 1 "MF-FSMF050X-2" H 2932 5545 50  0000 R CNN
+F 2 "ubmp:R_0603_1608Metric_Rounded" H 3050 5300 50  0001 L CNN
+F 3 "http://www.bourns.com/docs/Product-Datasheets/mffsmf.pdf" H 3000 5500 50  0001 C CNN
+	1    3000 5500
+	-1   0    0    1
+$EndComp
+Wire Wire Line
+	3000 5600 3000 5850
+Wire Wire Line
+	3000 5850 3050 5850
+$Comp
+L Device:R R1
+U 1 1 5AB8B470
+P 1750 4350
+F 0 "R1" V 1650 4350 50  0000 C CNN
+F 1 "100" V 1750 4350 50  0000 C CNN
+F 2 "ubmp:R_0402_1005Metric_Rounded" V 1680 4350 50  0001 C CNN
+F 3 "~" H 1750 4350 50  0001 C CNN
+	1    1750 4350
+	1    0    0    -1
+$EndComp
+Wire Wire Line
+	2700 4300 2350 4300
+Wire Wire Line
+	2350 4300 2350 4200
+Text Label 2500 4400 2    50   ~ 0
+BMP_SWCLK_TCK
+Wire Wire Line
+	2500 4400 2700 4400
+Wire Wire Line
+	2550 4500 2550 4550
+Connection ~ 2550 4500
+Wire Wire Line
+	2550 4500 2500 4500
+$Comp
+L Device:R R17
+U 1 1 5AB99A85
+P 8950 2650
+F 0 "R17" V 8850 2650 50  0000 C CNN
+F 1 "1.5k" V 8950 2650 50  0000 C CNN
+F 2 "ubmp:R_0402_1005Metric_Rounded" V 8880 2650 50  0001 C CNN
+F 3 "~" H 8950 2650 50  0001 C CNN
+	1    8950 2650
+	1    0    0    -1
+$EndComp
+$Comp
+L Device:R R18
+U 1 1 5AB99B2D
+P 9150 2650
+F 0 "R18" V 9050 2650 50  0000 C CNN
+F 1 "1.5k" V 9150 2650 50  0000 C CNN
+F 2 "ubmp:R_0402_1005Metric_Rounded" V 9080 2650 50  0001 C CNN
+F 3 "~" H 9150 2650 50  0001 C CNN
+	1    9150 2650
+	1    0    0    -1
+$EndComp
+$Comp
+L power:+3.3V #PWR01
+U 1 1 5AB99BF0
+P 8950 2500
+F 0 "#PWR01" H 8950 2350 50  0001 C CNN
+F 1 "+3.3V" V 8965 2628 50  0000 L CNN
+F 2 "" H 8950 2500 50  0001 C CNN
+F 3 "" H 8950 2500 50  0001 C CNN
+	1    8950 2500
+	1    0    0    -1
+$EndComp
+$Comp
+L power:GND #PWR026
+U 1 1 5AB99C87
+P 9150 2500
+F 0 "#PWR026" H 9150 2250 50  0001 C CNN
+F 1 "GND" H 9155 2327 50  0000 C CNN
+F 2 "" H 9150 2500 50  0001 C CNN
+F 3 "" H 9150 2500 50  0001 C CNN
+	1    9150 2500
+	-1   0    0    1
+$EndComp
+Wire Wire Line
+	9150 2800 9150 2900
+Wire Wire Line
+	9150 2900 8950 2900
+Wire Wire Line
+	8950 2900 8950 2800
+Wire Wire Line
+	8500 3100 8950 3100
+Wire Wire Line
+	8950 3100 8950 2900
+Connection ~ 8950 2900
+Text Label 8700 3100 0    50   ~ 0
+STLINK_AIN_1
+Wire Wire Line
+	1750 4550 1750 4500
+Wire Wire Line
+	1750 4550 2550 4550
+Wire Wire Line
+	2350 4200 1750 4200
+Text Label 1750 4200 0    50   ~ 0
+STLINK_SWDIO_IN
+Text Notes 1600 3950 0    50   ~ 0
+STLink compatibility
+Wire Notes Line
+	1950 4000 1950 4100
+Wire Notes Line
+	2200 4000 2200 4300
+Wire Notes Line
+	1600 4000 2350 4000
+Text Notes 9250 3000 0    50   ~ 0
+STLink compatibility
+$Comp
+L Device:R R19
+U 1 1 5ABBFC68
+P 2150 2800
+F 0 "R19" V 2050 2800 50  0000 C CNN
+F 1 "1.5k" V 2150 2800 50  0000 C CNN
+F 2 "ubmp:R_0402_1005Metric_Rounded" V 2080 2800 50  0001 C CNN
+F 3 "~" H 2150 2800 50  0001 C CNN
+	1    2150 2800
+	0    1    -1   0
+$EndComp
+$Comp
+L power:GND #PWR027
+U 1 1 5ABBFCC0
+P 2000 2800
+F 0 "#PWR027" H 2000 2550 50  0001 C CNN
+F 1 "GND" V 2005 2672 50  0000 R CNN
+F 2 "" H 2000 2800 50  0001 C CNN
+F 3 "" H 2000 2800 50  0001 C CNN
+	1    2000 2800
+	0    1    1    0
+$EndComp
+Text Label 2350 2800 0    50   ~ 0
+STM_ID2
+Wire Wire Line
+	2300 2800 2700 2800
+$Comp
+L power:GND #PWR0101
+U 1 1 5ABC82DD
+P 2700 3300
+F 0 "#PWR0101" H 2700 3050 50  0001 C CNN
+F 1 "GND" V 2705 3172 50  0000 R CNN
+F 2 "" H 2700 3300 50  0001 C CNN
+F 3 "" H 2700 3300 50  0001 C CNN
+	1    2700 3300
+	0    1    1    0
+$EndComp
 $EndSCHEMATC
