File: ubmp_v1_pcbusb.sch (KiCad schematic (older format))
At the start: 33 parts, among them J1 Conn_02x05_Counter_Clockwise, J2 USB_A, U1 STM32F103CBUx, U2 MIC5245-3.3, Y1 PRQC8.00CR1010V00L

Commit message: Bumped schematic date
Other:
- note added: "2018-03-27"
- note removed: "2018-02-16"
Changed lines of the file:
@@
 µBMP
 Text Notes 8150 7650 0    67   ~ 0
-2018-02-16
+2018-03-27
 Text Notes 10600 7650 0    67   ~ 0
 1.1

Commit message: Changed all 100 and 22 ohm resistors to ESD chips with built in resistors
Parts:
- removed R10, R11, R12, R13, R3, R4, R5: 100, ubmp:R_0402_1005Metric_Rounded, symbol Device:R
- removed R15, R16, R9: 22, ubmp:R_0402_1005Metric_Rounded, symbol Device:R
- added U3: NUF8401MNT4G, ubmp:DFN-16-1EP_1.6x4mm_P0.5mm, symbol Interface_ESD:NUF8401MNT4G
- added U4: NUF2042XV6T1G, ubmp:DFN-6-1EP_1.2x1.6mm_P0.5mm, symbol Interface_ESD:NUF2042XV6T1G
- renumbered R7 to R1, R8 to R2, R19 to R3, R14 to R4, R2 to R5
Connections:
- wire segments 98 -> 104
Other:
- note added: "1.2"
- note added: "2018-03-28"
- note removed: "1.1"
- note removed: "2018-03-27"
- note removed: "RST resistor is 22 Ohm to support board with small (<1.5k) pullup on RST"

Commit message: Split into hierarchical sheep
Parts:
- removed C1, C2, C3, C4, C7: 100n, ubmp:C_0402_1005Metric_Rounded, symbol Device:C_Small
- removed C5, C6: 4.7u, ubmp:C_0603_1608Metric_Rounded, symbol Device:C_Small
- removed D2: GREEN, ubmp:D_0603_1608Metric_Rounded, symbol Device:LED
- removed F1: MF-FSMF050X-2, ubmp:R_0603_1608Metric_Rounded, symbol Device:Polyfuse_Small
- removed J1: Conn_02x05_Counter_Clockwise, ubmp:2x5_2.54mm_side, symbol Connector_Generic:Conn_02x05_Counter_Clockwise
- removed R1, R2, R3, R4: 1.5k, ubmp:R_0402_1005Metric_Rounded, symbol Device:R
- removed R5: 470, ubmp:R_0402_1005Metric_Rounded, symbol Device:R
- removed TP1, TP2, TP3, TP4: Test_Point, TestPoint:TestPoint_Pad_D1.0mm, symbol Connector_Specialized:Test_Point
- removed U1: STM32F103CBUx, ubmp:QFN-48-1EP_7x7mm_P0.5mm_EP5.15x5.15mm, symbol MCU_ST_STM32:STM32F103CBUx
- removed U2: MIC5245-3.3, ubmp:SOT-23-5_Rounded, symbol Regulator_Linear:MIC5205-3.3
- removed U3: NUF8401MNT4G, ubmp:DFN-16-1EP_1.6x4mm_P0.5mm, symbol Interface_ESD:NUF8401MNT4G
- removed U4: NUF2042XV6T1G, ubmp:DFN-6-1EP_1.2x1.6mm_P0.5mm, symbol Interface_ESD:NUF2042XV6T1G
- removed Y1: PRQC8.00CR1010V00L, ubmp:Resonator_3pin_3.2x1.3mm, symbol Device:Resonator
Connections:
- net labels removed: +3.3V, BMP_RST, BMP_RSTo, BMP_RX, BMP_RXo, BMP_SWCLK_TCK, BMP_SWCLK_TCKo, BMP_SWDIO_TMS, BMP_SWDIO_TMSo, BMP_SWO, BMP_SWOo, BMP_TDI, BMP_TDIo, BMP_TDO, BMP_TDOo, BMP_TX, BMP_TXo, BOOT0, DM_P, DP_P, LED_STLINK, NRST, STM_ID, STM_ID2, SWCLK, SWDIO
- wire segments 104 -> 13
- no-connect marks 21 -> 0
Other:
- note removed: "MCO"
- note removed: "STLink V2 identifier (PC13 = 0)"
- note removed: "SWD Programming"

Commit message: Updated pinput
Changed lines of the file:
@@
 $EndDescr
 $Comp
-L power:+5V #PWR023
+L power:+5V #PWR01
 U 1 1 5A78C20D
-P 8450 4100
-F 0 "#PWR023" H 8450 3950 50  0001 C CNN
-F 1 "+5V" V 8465 4228 50  0000 L CNN
-F 2 "" H 8450 4100 50  0001 C CNN
-F 3 "" H 8450 4100 50  0001 C CNN
-	1    8450 4100
+P 6250 3950
+F 0 "#PWR01" H 6250 3800 50  0001 C CNN
+F 1 "+5V" V 6265 4078 50  0000 L CNN
+F 2 "" H 6250 3950 50  0001 C CNN
+F 3 "" H 6250 3950 50  0001 C CNN
+	1    6250 3950
 	0    -1   -1   0
 $EndComp
 $Comp
-L power:GND #PWR024
+L power:GND #PWR02
 U 1 1 5A78C254
-P 8950 3400
-F 0 "#PWR024" H 8950 3150 50  0001 C CNN
-F 1 "GND" H 8955 3227 50  0000 C CNN
-F 2 "" H 8950 3400 50  0001 C CNN
-F 3 "" H 8950 3400 50  0001 C CNN
-	1    8950 3400
+P 6750 3250
+F 0 "#PWR02" H 6750 3000 50  0001 C CNN
+F 1 "GND" H 6755 3077 50  0000 C CNN
+F 2 "" H 6750 3250 50  0001 C CNN
+F 3 "" H 6750 3250 50  0001 C CNN
+	1    6750 3250
 	-1   0    0    1
 $EndComp
 Wire Wire Line
-	8950 3400 8950 3450
+	6750 3250 6750 3300
 Wire Wire Line
-	8950 3450 8850 3450
+	6750 3300 6650 3300
 Wire Wire Line
-	8850 3450 8850 3500
-Connection ~ 8950 3450
+	6650 3300 6650 3350
+Connection ~ 6750 3300
 Wire Wire Line
-	8950 3450 8950 3500
-Text Label 8400 3900 0    50   ~ 0
+	6750 3300 6750 3350
+Text Label 6200 3750 0    50   ~ 0
 DP
-Text Label 8400 3800 0    50   ~ 0
+Text Label 6200 3650 0    50   ~ 0
 DM
 $Comp
 L Connector_Specialized:USB_A J2
 U 1 1 5A80B5EC
-P 8850 3900
-F 0 "J2" H 8906 4367 50  0000 C CNN
-F 1 "USB_A" H 8906 4276 50  0000 C CNN
-F 2 "usbpcb:USBPCB" H 9000 3850 50  0001 C CNN
-F 3 "" H 9000 3850 50  0001 C CNN
-	1    8850 3900
+P 6650 3750
+F 0 "J2" H 6706 4217 50  0000 C CNN
+F 1 "USB_A" H 6706 4126 50  0000 C CNN
+F 2 "usbpcb:USBPCB" H 6800 3700 50  0001 C CNN
+F 3 "" H 6800 3700 50  0001 C CNN
+	1    6650 3750
 	-1   0    0    1
 $EndComp
 Wire Wire Line
-	8450 4100 8500 4100
+	6250 3950 6300 3950
 $Comp
 L power:PWR_FLAG #FLG01
 U 1 1 5A8464BC
-P 8500 4100
-F 0 "#FLG01" H 8500 4175 50  0001 C CNN
-F 1 "PWR_FLAG" H 8500 4274 50  0000 C CNN
-F 2 "" H 8500 4100 50  0001 C CNN
-F 3 "" H 8500 4100 50  0001 C CNN
-	1    8500 4100
+P 6300 3950
+F 0 "#FLG01" H 6300 4025 50  0001 C CNN
+F 1 "PWR_FLAG" H 6300 4124 50  0000 C CNN
+F 2 "" H 6300 3950 50  0001 C CNN
+F 3 "" H 6300 3950 50  0001 C CNN
+	1    6300 3950
 	-1   0    0    1
 $EndComp
-Connection ~ 8500 4100
+Connection ~ 6300 3950
 $Comp
 L power:PWR_FLAG #FLG02
 U 1 1 5A84681F
-P 8850 3450
-F 0 "#FLG02" H 8850 3525 50  0001 C CNN
-F 1 "PWR_FLAG" V 8850 3578 50  0000 L CNN
-F 2 "" H 8850 3450 50  0001 C CNN
-F 3 "" H 8850 3450 50  0001 C CNN
-	1    8850 3450
+P 6650 3300
+F 0 "#FLG02" H 6650 3375 50  0001 C CNN
+F 1 "PWR_FLAG" V 6650 3428 50  0000 L CNN
+F 2 "" H 6650 3300 50  0001 C CNN
+F 3 "" H 6650 3300 50  0001 C CNN
+	1    6650 3300
 	0    -1   -1   0
 $EndComp
-Connection ~ 8850 3450
+Connection ~ 6650 3300
 $Comp
 L Graphic:Logo_Open_Hardware_Small #LOGO1
@@
 Design available at: github.com/korken89/micro-bmp
 Wire Wire Line
-	8500 4100 8550 4100
+	6300 3950 6350 3950
 $Sheet
-S 6900 3500 550  600
+S 4700 3350 550  600
 U 5ABD6923
 F0 "bmp_core" 50
 F1 "bmp_core.sch" 50
-F2 "5V" I R 7450 4000 50
-F3 "DP" I R 7450 3900 50
-F4 "DM" I R 7450 3800 50
-F5 "GND" I R 7450 3700 50
+F2 "5V" I R 5250 3850 50
+F3 "DP" I R 5250 3750 50
+F4 "DM" I R 5250 3650 50
+F5 "GND" I R 5250 3550 50
 $EndSheet
 Wire Wire Line
-	8500 4100 8500 4000
+	6300 3950 6300 3850
 Wire Wire Line
-	8500 4000 7450 4000
+	6300 3850 5250 3850
 Wire Wire Line
-	8550 3900 7450 3900
+	6350 3750 5250 3750
 Wire Wire Line
-	8550 3800 7450 3800
+	6350 3650 5250 3650
 Wire Wire Line
-	8850 3500 7600 3500
+	6650 3350 5400 3350
 Wire Wire Line
-	7600 3500 7600 3700
+	5400 3350 5400 3550
 Wire Wire Line
-	7600 3700 7450 3700
-Connection ~ 8850 3500
+	5400 3550 5250 3550
+Connection ~ 6650 3350
 $EndSCHEMATC

Commit message: Updated PCB USB version
Parts:
- J2: footprint usbpcb:USBPCB -> usb:USBPCB
Connections:
- wire segments 13 -> 12
Other:
- note added: "1.1"
- note added: "2018-03-27"
- note removed: "1.2"
- note removed: "2018-03-28"
Changed lines of the file:
@@
 L power:+5V #PWR01
 U 1 1 5A78C20D
-P 6250 3950
-F 0 "#PWR01" H 6250 3800 50  0001 C CNN
-F 1 "+5V" V 6265 4078 50  0000 L CNN
-F 2 "" H 6250 3950 50  0001 C CNN
-F 3 "" H 6250 3950 50  0001 C CNN
-	1    6250 3950
+P 6150 4150
+F 0 "#PWR01" H 6150 4000 50  0001 C CNN
+F 1 "+5V" V 6165 4278 50  0000 L CNN
+F 2 "" H 6150 4150 50  0001 C CNN
+F 3 "" H 6150 4150 50  0001 C CNN
+	1    6150 4150
 	0    -1   -1   0
 $EndComp
@@
 L power:GND #PWR02
 U 1 1 5A78C254
-P 6750 3250
-F 0 "#PWR02" H 6750 3000 50  0001 C CNN
-F 1 "GND" H 6755 3077 50  0000 C CNN
-F 2 "" H 6750 3250 50  0001 C CNN
-F 3 "" H 6750 3250 50  0001 C CNN
-	1    6750 3250
+P 6600 3450
+F 0 "#PWR02" H 6600 3200 50  0001 C CNN
+F 1 "GND" H 6605 3277 50  0000 C CNN
+F 2 "" H 6600 3450 50  0001 C CNN
+F 3 "" H 6600 3450 50  0001 C CNN
+	1    6600 3450
 	-1   0    0    1
 $EndComp
 Wire Wire Line
-	6750 3250 6750 3300
+	6600 3450 6600 3500
 Wire Wire Line
-	6750 3300 6650 3300
+	6600 3500 6500 3500
 Wire Wire Line
-	6650 3300 6650 3350
-Connection ~ 6750 3300
+	6500 3500 6500 3550
+Connection ~ 6600 3500
 Wire Wire Line
-	6750 3300 6750 3350
-Text Label 6200 3750 0    50   ~ 0
+	6600 3500 6600 3550
+Text Label 6050 3950 0    50   ~ 0
 DP
-Text Label 6200 3650 0    50   ~ 0
+Text Label 6050 3850 0    50   ~ 0
 DM
 $Comp
 L Connector_Specialized:USB_A J2
 U 1 1 5A80B5EC
-P 6650 3750
-F 0 "J2" H 6706 4217 50  0000 C CNN
-F 1 "USB_A" H 6706 4126 50  0000 C CNN
-F 2 "usbpcb:USBPCB" H 6800 3700 50  0001 C CNN
-F 3 "" H 6800 3700 50  0001 C CNN
-	1    6650 3750
+P 6500 3950
+F 0 "J2" H 6556 4417 50  0000 C CNN
+F 1 "USB_A" H 6556 4326 50  0000 C CNN
+F 2 "usb:USBPCB" H 6650 3900 50  0001 C CNN
+F 3 "" H 6650 3900 50  0001 C CNN
+	1    6500 3950
 	-1   0    0    1
 $EndComp
 Wire Wire Line
-	6250 3950 6300 3950
+	6150 4150 6200 4150
 $Comp
 L power:PWR_FLAG #FLG01
 U 1 1 5A8464BC
-P 6300 3950
-F 0 "#FLG01" H 6300 4025 50  0001 C CNN
-F 1 "PWR_FLAG" H 6300 4124 50  0000 C CNN
-F 2 "" H 6300 3950 50  0001 C CNN
-F 3 "" H 6300 3950 50  0001 C CNN
-	1    6300 3950
+P 6150 4150
+F 0 "#FLG01" H 6150 4225 50  0001 C CNN
+F 1 "PWR_FLAG" H 6150 4324 50  0000 C CNN
+F 2 "" H 6150 4150 50  0001 C CNN
+F 3 "" H 6150 4150 50  0001 C CNN
+	1    6150 4150
 	-1   0    0    1
 $EndComp
-Connection ~ 6300 3950
+Connection ~ 6150 4150
 $Comp
 L power:PWR_FLAG #FLG02
 U 1 1 5A84681F
-P 6650 3300
-F 0 "#FLG02" H 6650 3375 50  0001 C CNN
-F 1 "PWR_FLAG" V 6650 3428 50  0000 L CNN
-F 2 "" H 6650 3300 50  0001 C CNN
-F 3 "" H 6650 3300 50  0001 C CNN
-	1    6650 3300
+P 6500 3500
+F 0 "#FLG02" H 6500 3575 50  0001 C CNN
+F 1 "PWR_FLAG" V 6500 3628 50  0000 L CNN
+F 2 "" H 6500 3500 50  0001 C CNN
+F 3 "" H 6500 3500 50  0001 C CNN
+	1    6500 3500
 	0    -1   -1   0
 $EndComp
-Connection ~ 6650 3300
+Connection ~ 6500 3500
 $Comp
 L Graphic:Logo_Open_Hardware_Small #LOGO1
@@
 µBMP
 Text Notes 8150 7650 0    67   ~ 0
-2018-03-28
+2018-03-27
 Text Notes 10600 7650 0    67   ~ 0
-1.2
+1.1
 Text Notes 7100 6850 0    79   ~ 0
 Note that this board is designed to work with the \nSTLink V2 version of Black Magic Probe firmware.
 Text Notes 7100 7050 0    79   ~ 0
 Design available at: github.com/korken89/micro-bmp
-Wire Wire Line
-	6300 3950 6350 3950
 $Sheet
-S 4700 3350 550  600
-U 5ABD6923
+S 4750 3650 700  500
+U 5ABFD4E7
 F0 "bmp_core" 50
 F1 "bmp_core.sch" 50
-F2 "5V" I R 5250 3850 50
-F3 "DP" I R 5250 3750 50
-F4 "DM" I R 5250 3650 50
-F5 "GND" I R 5250 3550 50
+F2 "5V" I R 5450 4050 50
+F3 "DP" I R 5450 3950 50
+F4 "DM" I R 5450 3850 50
+F5 "GND" I R 5450 3750 50
 $EndSheet
 Wire Wire Line
-	6300 3950 6300 3850
+	6200 3950 5450 3950
 Wire Wire Line
-	6300 3850 5250 3850
+	5450 3850 6200 3850
 Wire Wire Line
-	6350 3750 5250 3750
+	6500 3550 5600 3550
 Wire Wire Line
-	6350 3650 5250 3650
+	5600 3550 5600 3750
 Wire Wire Line
-	6650 3350 5400 3350
+	5600 3750 5450 3750
+Connection ~ 6500 3550
 Wire Wire Line
-	5400 3350 5400 3550
+	6150 4150 6150 4050
 Wire Wire Line
-	5400 3550 5250 3550
-Connection ~ 6650 3350
+	6150 4050 5450 4050
 $EndSCHEMATC
