File: bmp_core.sch (KiCad schematic (older format))
At the start: 24 parts, among them J1 Conn_02x05_Counter_Clockwise, U1 NUF8401MNT4G, U2 MIC5245-3.3, U3 STM32F103CBUx, U4 NUF2042XV6T1G, Y1 PRQC8.00CR1010V00L

Commit message: Updated pinput
Changed lines of the file:
@@
 Text Label 5000 6050 0    50   ~ 0
 BMP_TDOo
+Text Label 5000 6150 0    50   ~ 0
+BMP_TDIo
 Text Label 4050 6150 2    50   ~ 0
-BMP_TDIo
-Text Label 5000 6150 0    50   ~ 0
 BMP_RSTo
 Text Label 4050 6250 2    50   ~ 0

Commit message: Moved libs to external repo
Parts:
- C1, C3, C4, C6, C7: footprint ubmp:C_0402_1005Metric_Rounded -> passive:C_0402_1005Metric_Rounded
- C2, C5: footprint ubmp:C_0603_1608Metric_Rounded -> passive:C_0603_1608Metric_Rounded
- D1: footprint ubmp:D_0603_1608Metric_Rounded -> passive:D_0603_1608Metric_Rounded
- F1: footprint ubmp:R_0603_1608Metric_Rounded -> passive:R_0603_1608Metric_Rounded
- J1: footprint ubmp:2x5_2.54mm_side -> connectors:2x5_2.54mm_side
- R1, R2, R3, R4, R5: footprint ubmp:R_0402_1005Metric_Rounded -> passive:R_0402_1005Metric_Rounded
- U1: footprint ubmp:DFN-16-1EP_1.6x4mm_P0.5mm -> dfn:DFN-16-1EP_1.6x4mm_P0.5mm; symbol Interface_ESD:NUF8401MNT4G -> interface_esd:NUF8401MNT4G
- U2: footprint ubmp:SOT-23-5_Rounded -> sot:SOT-23-5
- U3: footprint ubmp:QFN-48-1EP_7x7mm_P0.5mm_EP5.15x5.15mm -> qfn:QFN-48-1EP_7x7mm_P0.5mm_EP5.15x5.15mm
- U4: footprint ubmp:DFN-6-1EP_1.2x1.6mm_P0.5mm -> dfn:DFN-6-1EP_1.2x1.6mm_P0.5mm; symbol Interface_ESD:NUF2042XV6T1G -> interface_esd:NUF2042XV6T1G
- Y1: footprint ubmp:Resonator_3pin_3.2x1.3mm -> crystals:Resonator_3pin_3.2x1.3mm
Changed lines of the file:
@@
 F 0 "U3" H 2800 4950 50  0000 C CNN
 F 1 "STM32F103CBUx" H 8050 4950 50  0000 C CNN
-F 2 "ubmp:QFN-48-1EP_7x7mm_P0.5mm_EP5.15x5.15mm" H 8350 4875 50  0001 R TNN
+F 2 "qfn:QFN-48-1EP_7x7mm_P0.5mm_EP5.15x5.15mm" H 8350 4875 50  0001 R TNN
 F 3 "http://www.st.com/st-web-ui/static/active/en/resource/technical/document/datasheet/CD00161566.pdf" H 5550 3200 50  0001 C CNN
 	1    5550 3200
@@
 F 0 "C7" H 4542 1146 50  0000 L CNN
 F 1 "100n" H 4542 1055 50  0000 L CNN
-F 2 "ubmp:C_0402_1005Metric_Rounded" H 4450 1100 50  0001 C CNN
+F 2 "passive:C_0402_1005Metric_Rounded" H 4450 1100 50  0001 C CNN
 F 3 "~" H 4450 1100 50  0001 C CNN
 	1    4450 1100
@@
 F 0 "C6" H 4192 1146 50  0000 L CNN
 F 1 "100n" H 4192 1055 50  0000 L CNN
-F 2 "ubmp:C_0402_1005Metric_Rounded" H 4100 1100 50  0001 C CNN
+F 2 "passive:C_0402_1005Metric_Rounded" H 4100 1100 50  0001 C CNN
 F 3 "~" H 4100 1100 50  0001 C CNN
 	1    4100 1100
@@
 F 0 "C4" H 3842 1146 50  0000 L CNN
 F 1 "100n" H 3842 1055 50  0000 L CNN
-F 2 "ubmp:C_0402_1005Metric_Rounded" H 3750 1100 50  0001 C CNN
+F 2 "passive:C_0402_1005Metric_Rounded" H 3750 1100 50  0001 C CNN
 F 3 "~" H 3750 1100 50  0001 C CNN
 	1    3750 1100
@@
 F 0 "C3" H 3492 1146 50  0000 L CNN
 F 1 "100n" H 3492 1055 50  0000 L CNN
-F 2 "ubmp:C_0402_1005Metric_Rounded" H 3400 1100 50  0001 C CNN
+F 2 "passive:C_0402_1005Metric_Rounded" H 3400 1100 50  0001 C CNN
 F 3 "~" H 3400 1100 50  0001 C CNN
 	1    3400 1100
@@
 F 0 "Y1" V 1204 2311 50  0000 L CNN
 F 1 "PRQC8.00CR1010V00L" V 1295 2311 50  0000 L CNN
-F 2 "ubmp:Resonator_3pin_3.2x1.3mm" H 1225 2200 50  0001 C CNN
+F 2 "crystals:Resonator_3pin_3.2x1.3mm" H 1225 2200 50  0001 C CNN
 F 3 "~" H 1225 2200 50  0001 C CNN
 	1    1250 2200
@@
 F 0 "U2" H 3250 7392 50  0000 C CNN
 F 1 "MIC5245-3.3" H 3250 7301 50  0000 C CNN
-F 2 "ubmp:SOT-23-5_Rounded" H 3250 7375 50  0001 C CNN
+F 2 "sot:SOT-23-5" H 3250 7375 50  0001 C CNN
 F 3 "http://ww1.microchip.com/downloads/en/devicedoc/mic5205.pdf" H 3250 7050 50  0001 C CNN
 	1    3250 7050
@@
 F 0 "C2" H 2692 7146 50  0000 L CNN
 F 1 "4.7u" H 2692 7055 50  0000 L CNN
-F 2 "ubmp:C_0603_1608Metric_Rounded" H 2600 7100 50  0001 C CNN
+F 2 "passive:C_0603_1608Metric_Rounded" H 2600 7100 50  0001 C CNN
 F 3 "~" H 2600 7100 50  0001 C CNN
 	1    2600 7100
@@
 F 0 "C5" H 3842 7146 50  0000 L CNN
 F 1 "4.7u" H 3842 7055 50  0000 L CNN
-F 2 "ubmp:C_0603_1608Metric_Rounded" H 3750 7100 50  0001 C CNN
+F 2 "passive:C_0603_1608Metric_Rounded" H 3750 7100 50  0001 C CNN
 F 3 "~" H 3750 7100 50  0001 C CNN
 	1    3750 7100
@@
 F 0 "R1" V 2000 2000 50  0000 C CNN
 F 1 "1.5k" V 2100 2000 50  0000 C CNN
-F 2 "ubmp:R_0402_1005Metric_Rounded" V 2030 2000 50  0001 C CNN
+F 2 "passive:R_0402_1005Metric_Rounded" V 2030 2000 50  0001 C CNN
 F 3 "~" H 2100 2000 50  0001 C CNN
 	1    2100 2000
@@
 F 0 "J1" H 4500 6375 50  0000 C CNN
 F 1 "Conn_02x05_Counter_Clockwise" H 4500 6376 50  0001 C CNN
-F 2 "ubmp:2x5_2.54mm_side" H 4450 6050 50  0001 C CNN
+F 2 "connectors:2x5_2.54mm_side" H 4450 6050 50  0001 C CNN
 F 3 "~" H 4450 6050 50  0001 C CNN
 	1    4450 6050
@@
 F 0 "R2" V 2000 2700 50  0000 C CNN
 F 1 "1.5k" V 2100 2700 50  0000 C CNN
-F 2 "ubmp:R_0402_1005Metric_Rounded" V 2030 2700 50  0001 C CNN
+F 2 "passive:R_0402_1005Metric_Rounded" V 2030 2700 50  0001 C CNN
 F 3 "~" H 2100 2700 50  0001 C CNN
 	1    2100 2700
@@
 F 0 "D1" H 9750 1550 50  0000 C CNN
 F 1 "GREEN" H 9750 1300 50  0000 C CNN
-F 2 "ubmp:D_0603_1608Metric_Rounded" H 9750 1450 50  0001 C CNN
+F 2 "passive:D_0603_1608Metric_Rounded" H 9750 1450 50  0001 C CNN
 F 3 "~" H 9750 1450 50  0001 C CNN
 	1    9750 1450
@@
 F 0 "R5" V 9950 1450 50  0000 C CNN
 F 1 "470" V 10050 1450 50  0000 C CNN
-F 2 "ubmp:R_0402_1005Metric_Rounded" V 9980 1450 50  0001 C CNN
+F 2 "passive:R_0402_1005Metric_Rounded" V 9980 1450 50  0001 C CNN
 F 3 "~" H 10050 1450 50  0001 C CNN
 	1    10050 1450
@@
 F 0 "R4" V 9700 3650 50  0000 C CNN
 F 1 "1.5k" V 9800 3650 50  0000 C CNN
-F 2 "ubmp:R_0402_1005Metric_Rounded" V 9730 3650 50  0001 C CNN
+F 2 "passive:R_0402_1005Metric_Rounded" V 9730 3650 50  0001 C CNN
 F 3 "~" H 9800 3650 50  0001 C CNN
 	1    9800 3650
@@
 F 0 "F1" H 4132 5454 50  0000 R CNN
 F 1 "MF-FSMF050X-2" H 4132 5545 50  0000 R CNN
-F 2 "ubmp:R_0603_1608Metric_Rounded" H 4250 5300 50  0001 L CNN
+F 2 "passive:R_0603_1608Metric_Rounded" H 4250 5300 50  0001 L CNN
 F 3 "http://www.bourns.com/docs/Product-Datasheets/mffsmf.pdf" H 4200 5500 50  0001 C CNN
 	1    4200 5500
@@
 F 0 "R3" V 2000 2800 50  0000 C CNN
 F 1 "1.5k" V 2100 2800 50  0000 C CNN
-F 2 "ubmp:R_0402_1005Metric_Rounded" V 2030 2800 50  0001 C CNN
+F 2 "passive:R_0402_1005Metric_Rounded" V 2030 2800 50  0001 C CNN
 F 3 "~" H 2100 2800 50  0001 C CNN
 	1    2100 2800
@@
 F 0 "C1" H 2242 1846 50  0000 L CNN
 F 1 "100n" H 2242 1755 50  0000 L CNN
-F 2 "ubmp:C_0402_1005Metric_Rounded" H 2150 1800 50  0001 C CNN
+F 2 "passive:C_0402_1005Metric_Rounded" H 2150 1800 50  0001 C CNN
 F 3 "~" H 2150 1800 50  0001 C CNN
 	1    2150 1800
@@
 NoConn ~ 8450 3100
 $Comp
-L Interface_ESD:NUF2042XV6T1G U4
+L interface_esd:NUF2042XV6T1G U4
 U 1 1 5ABD71A7
 P 9800 4200
 F 0 "U4" H 9825 3885 50  0000 C CNN
 F 1 "NUF2042XV6T1G" H 9825 3976 50  0000 C CNN
-F 2 "ubmp:DFN-6-1EP_1.2x1.6mm_P0.5mm" H 9650 4150 50  0001 C CNN
+F 2 "dfn:DFN-6-1EP_1.2x1.6mm_P0.5mm" H 9650 4150 50  0001 C CNN
 F 3 "http://www.onsemi.com/pub/Collateral/NUF2030XV6-D.PDF" H 9800 3900 50  0001 C CNN
 	1    9800 4200
@@
 $EndComp
 $Comp
-L Interface_ESD:NUF8401MNT4G U1
+L interface_esd:NUF8401MNT4G U1
 U 1 1 5ABD71AE
 P 1750 5500
 F 0 "U1" H 1925 5675 50  0000 C CNN
 F 1 "NUF8401MNT4G" H 1925 5584 50  0000 C CNN
-F 2 "ubmp:DFN-16-1EP_1.6x4mm_P0.5mm" H 1750 5350 50  0001 C CNN
+F 2 "dfn:DFN-16-1EP_1.6x4mm_P0.5mm" H 1750 5350 50  0001 C CNN
 F 3 "http://www.onsemi.com/pub/Collateral/NUF8401MN-D.PDF" H 1950 4450 50  0001 C CNN
 	1    1750 5500

Commit message: Updated components + libs and changed to 1.5k resistor arrary
Parts:
- removed R1, R2, R3, R4: 1.5k, passive:R_0402_1005Metric_Rounded, symbol Device:R
- added RN1: 1.5k, passive:R_Array_Convex_4x0402, symbol Device:R_Pack04
- D1: footprint passive:D_0603_1608Metric_Rounded -> leds:LEDC1608X60
- renumbered R5 to R1
Connections:
- net labels removed: STM_ID2
- wire segments 98 -> 94
- no-connect marks 21 -> 23
Changed lines of the file:
@@
 EESchema Schematic File Version 4
+LIBS:ubmp_v1-cache
 EELAYER 26 0
 EELAYER END
@@
 $EndComp
 $Comp
-L Device:R R1
-U 1 1 5ABD7073
-P 2100 2000
-F 0 "R1" V 2000 2000 50  0000 C CNN
-F 1 "1.5k" V 2100 2000 50  0000 C CNN
-F 2 "passive:R_0402_1005Metric_Rounded" V 2030 2000 50  0001 C CNN
-F 3 "~" H 2100 2000 50  0001 C CNN
-	1    2100 2000
-	0    1    1    0
-$EndComp
-$Comp
 L power:GND #PWR04
 U 1 1 5ABD707A
-P 1950 2000
-F 0 "#PWR04" H 1950 1750 50  0001 C CNN
-F 1 "GND" V 1955 1872 50  0000 R CNN
-F 2 "" H 1950 2000 50  0001 C CNN
-F 3 "" H 1950 2000 50  0001 C CNN
-	1    1950 2000
-	0    1    1    0
+P 10050 2400
+F 0 "#PWR04" H 10050 2150 50  0001 C CNN
+F 1 "GND" V 10055 2272 50  0000 R CNN
+F 2 "" H 10050 2400 50  0001 C CNN
+F 3 "" H 10050 2400 50  0001 C CNN
+	1    10050 2400
+	0    -1   -1   0
 $EndComp
 Text Label 1550 6250 2    50   ~ 0
@@
 	1650 6150 1550 6150
 $Comp
-L Device:R R2
-U 1 1 5ABD70FF
-P 2100 2700
-F 0 "R2" V 2000 2700 50  0000 C CNN
-F 1 "1.5k" V 2100 2700 50  0000 C CNN
-F 2 "passive:R_0402_1005Metric_Rounded" V 2030 2700 50  0001 C CNN
-F 3 "~" H 2100 2700 50  0001 C CNN
-	1    2100 2700
-	0    1    1    0
-$EndComp
-$Comp
 L power:GND #PWR05
 U 1 1 5ABD7106
-P 1950 2700
-F 0 "#PWR05" H 1950 2450 50  0001 C CNN
-F 1 "GND" V 1955 2572 50  0000 R CNN
-F 2 "" H 1950 2700 50  0001 C CNN
-F 3 "" H 1950 2700 50  0001 C CNN
-	1    1950 2700
-	0    1    1    0
+P 10050 2600
+F 0 "#PWR05" H 10050 2350 50  0001 C CNN
+F 1 "GND" V 10055 2472 50  0000 R CNN
+F 2 "" H 10050 2600 50  0001 C CNN
+F 3 "" H 10050 2600 50  0001 C CNN
+	1    10050 2600
+	0    -1   -1   0
 $EndComp
 Text Notes 750  2600 0    50   ~ 0
@@
 F 0 "D1" H 9750 1550 50  0000 C CNN
 F 1 "GREEN" H 9750 1300 50  0000 C CNN
-F 2 "passive:D_0603_1608Metric_Rounded" H 9750 1450 50  0001 C CNN
+F 2 "leds:LEDC1608X60" H 9750 1450 50  0001 C CNN
 F 3 "~" H 9750 1450 50  0001 C CNN
 	1    9750 1450
@@
 $EndComp
 $Comp
-L Device:R R5
+L Device:R R1
 U 1 1 5ABD711F
 P 10050 1450
-F 0 "R5" V 9950 1450 50  0000 C CNN
+F 0 "R1" V 9950 1450 50  0000 C CNN
 F 1 "470" V 10050 1450 50  0000 C CNN
 F 2 "passive:R_0402_1005Metric_Rounded" V 9980 1450 50  0001 C CNN
@@
 Text Label 8650 4000 0    50   ~ 0
 LED_STLINK
-$Comp
-L Device:R R4
-U 1 1 5ABD7129
-P 9800 3650
-F 0 "R4" V 9700 3650 50  0000 C CNN
-F 1 "1.5k" V 9800 3650 50  0000 C CNN
-F 2 "passive:R_0402_1005Metric_Rounded" V 9730 3650 50  0001 C CNN
-F 3 "~" H 9800 3650 50  0001 C CNN
-	1    9800 3650
-	0    1    1    0
-$EndComp
 Wire Wire Line
 	10600 4200 10400 4200
@@
 L power:+3.3V #PWR027
 U 1 1 5ABD7131
-P 9950 3650
-F 0 "#PWR027" H 9950 3500 50  0001 C CNN
-F 1 "+3.3V" V 9965 3778 50  0000 L CNN
-F 2 "" H 9950 3650 50  0001 C CNN
-F 3 "" H 9950 3650 50  0001 C CNN
-	1    9950 3650
-	0    1    1    0
+P 9650 2700
+F 0 "#PWR027" H 9650 2550 50  0001 C CNN
+F 1 "+3.3V" V 9665 2828 50  0000 L CNN
+F 2 "" H 9650 2700 50  0001 C CNN
+F 3 "" H 9650 2700 50  0001 C CNN
+	1    9650 2700
+	0    -1   -1   0
 $EndComp
 Wire Wire Line
@@
 Text Label 2300 1800 0    50   ~ 0
 NRST
-Text Label 2300 2000 0    50   ~ 0
+Text Label 2450 2000 2    50   ~ 0
 BOOT0
 Wire Wire Line
 	2250 1800 2650 1800
 Wire Wire Line
-	2250 2000 2650 2000
-Wire Wire Line
-	2250 2700 2650 2700
-Text Label 2300 2700 0    50   ~ 0
+	2450 2000 2650 2000
+Wire Wire Line
+	2450 2700 2650 2700
+Text Label 2450 2700 2    50   ~ 0
 STM_ID
 Text Label 2350 6250 0    50   ~ 0
@@
 	4200 5850 4250 5850
 $Comp
-L Device:R R3
-U 1 1 5ABD7182
-P 2100 2800
-F 0 "R3" V 2000 2800 50  0000 C CNN
-F 1 "1.5k" V 2100 2800 50  0000 C CNN
-F 2 "passive:R_0402_1005Metric_Rounded" V 2030 2800 50  0001 C CNN
-F 3 "~" H 2100 2800 50  0001 C CNN
-	1    2100 2800
-	0    1    -1   0
-$EndComp
-$Comp
-L power:GND #PWR06
-U 1 1 5ABD7189
-P 1950 2800
-F 0 "#PWR06" H 1950 2550 50  0001 C CNN
-F 1 "GND" V 1955 2672 50  0000 R CNN
-F 2 "" H 1950 2800 50  0001 C CNN
-F 3 "" H 1950 2800 50  0001 C CNN
-	1    1950 2800
-	0    1    1    0
-$EndComp
-Text Label 2300 2800 0    50   ~ 0
-STM_ID2
-Wire Wire Line
-	2250 2800 2650 2800
-$Comp
 L Device:C_Small C1
 U 1 1 5ABD7191
@@
 	9250 4100 9500 4100
 Wire Wire Line
-	8450 4300 9150 4300
-Wire Wire Line
 	10150 4300 10600 4300
 Wire Wire Line
@@
 	0    1    1    0
 $EndComp
-Wire Wire Line
-	9150 3650 9150 4300
-Wire Wire Line
-	9150 3650 9650 3650
-Connection ~ 9150 4300
-Wire Wire Line
-	9150 4300 9500 4300
 $Comp
 L power:GND #PWR08
@@
 Text HLabel 10600 4400 2    50   Input ~ 0
 GND
+$Comp
+L Device:R_Pack04 RN1
+U 1 1 5ABF7111
+P 9850 2600
+F 0 "RN1" V 9433 2600 50  0000 C CNN
+F 1 "1.5k" V 9524 2600 50  0000 C CNN
+F 2 "passive:R_Array_Convex_4x0402" V 10125 2600 50  0001 C CNN
+F 3 "~" H 9850 2600 50  0001 C CNN
+	1    9850 2600
+	0    1    1    0
+$EndComp
+Text Label 9650 2400 2    50   ~ 0
+STM_ID
+Text Label 9650 2600 2    50   ~ 0
+BOOT0
+Text Label 10050 2700 0    50   ~ 0
+DP_P
+Wire Wire Line
+	8450 4300 9500 4300
+NoConn ~ 2650 2800
+$Comp
+L power:GND #PWR06
+U 1 1 5ABD7189
+P 10050 2500
+F 0 "#PWR06" H 10050 2250 50  0001 C CNN
+F 1 "GND" V 10055 2372 50  0000 R CNN
+F 2 "" H 10050 2500 50  0001 C CNN
+F 3 "" H 10050 2500 50  0001 C CNN
+	1    10050 2500
+	0    -1   -1   0
+$EndComp
+NoConn ~ 9650 2500
 $EndSCHEMATC

Commit message: Updated part numbers
Parts:
- D1: value GREEN -> LTST-C191KGKT
- J1: value Conn_02x05_Counter_Clockwise -> M20-9760542
- RN1: value 1.5k -> EXB-28V152JX
- U2: value MIC5245-3.3 -> MIC5245-3.3YM5
- U3: value STM32F103CBUx -> STM32F103CBU6
Connections:
- wire segments 94 -> 92
Changed lines of the file:
@@
 P 5550 3200
 F 0 "U3" H 2800 4950 50  0000 C CNN
-F 1 "STM32F103CBUx" H 8050 4950 50  0000 C CNN
+F 1 "STM32F103CBU6" H 8050 4950 50  0000 C CNN
 F 2 "qfn:QFN-48-1EP_7x7mm_P0.5mm_EP5.15x5.15mm" H 8350 4875 50  0001 R TNN
 F 3 "http://www.st.com/st-web-ui/static/active/en/resource/technical/document/datasheet/CD00161566.pdf" H 5550 3200 50  0001 C CNN
@@
 P 3250 7050
 F 0 "U2" H 3250 7392 50  0000 C CNN
-F 1 "MIC5245-3.3" H 3250 7301 50  0000 C CNN
+F 1 "MIC5245-3.3YM5" H 3250 7301 50  0000 C CNN
 F 2 "sot:SOT-23-5" H 3250 7375 50  0001 C CNN
 F 3 "http://ww1.microchip.com/downloads/en/devicedoc/mic5205.pdf" H 3250 7050 50  0001 C CNN
@@
 Text Label 10450 4300 0    50   ~ 0
 DP
-Text Label 10450 4200 0    50   ~ 0
+Text Label 10450 4100 0    50   ~ 0
 DM
 Wire Wire Line
@@
 P 4450 6050
 F 0 "J1" H 4500 6375 50  0000 C CNN
-F 1 "Conn_02x05_Counter_Clockwise" H 4500 6376 50  0001 C CNN
+F 1 "M20-9760542" H 4500 5750 50  0000 C CNN
 F 2 "connectors:2x5_2.54mm_side" H 4450 6050 50  0001 C CNN
-F 3 "~" H 4450 6050 50  0001 C CNN
+F 3 "https://cdn.harwin.com/pdfs/M20-976.pdf" H 4450 6050 50  0001 C CNN
 	1    4450 6050
 	1    0    0    -1
@@
 P 9750 1450
 F 0 "D1" H 9750 1550 50  0000 C CNN
-F 1 "GREEN" H 9750 1300 50  0000 C CNN
+F 1 "LTST-C191KGKT" H 9750 1300 50  0000 C CNN
 F 2 "leds:LEDC1608X60" H 9750 1450 50  0001 C CNN
 F 3 "~" H 9750 1450 50  0001 C CNN
@@
 Text Label 8650 4000 0    50   ~ 0
 LED_STLINK
-Wire Wire Line
-	10600 4200 10400 4200
 $Comp
 L power:+3.3V #PWR027
@@
 Wire Wire Line
 	10150 4300 10600 4300
-Wire Wire Line
-	10150 4100 10400 4100
-Wire Wire Line
-	10400 4100 10400 4200
 $Comp
 L power:+5V #PWR028
@@
 Text HLabel 10600 4300 2    50   Input ~ 0
 DP
-Text HLabel 10600 4200 2    50   Input ~ 0
+Text HLabel 10600 4100 2    50   Input ~ 0
 DM
 Text HLabel 10600 4400 2    50   Input ~ 0
@@
 P 9850 2600
 F 0 "RN1" V 9433 2600 50  0000 C CNN
-F 1 "1.5k" V 9524 2600 50  0000 C CNN
+F 1 "EXB-28V152JX" V 9524 2600 50  0000 C CNN
 F 2 "passive:R_Array_Convex_4x0402" V 10125 2600 50  0001 C CNN
 F 3 "~" H 9850 2600 50  0001 C CNN
@@
 $EndComp
 NoConn ~ 9650 2500
+Wire Wire Line
+	10150 4100 10600 4100
 $EndSCHEMATC

Commit message: Bumped schematic date and added value to resistor array
Other:
- note added: "1.5k"
- note added: "2018-04-03"
- note removed: "2018-03-28"
Changed lines of the file:
@@
 µBMP
 Text Notes 8100 7650 0    67   ~ 0
-2018-03-28
+2018-04-03
 Text Notes 10550 7650 0    67   ~ 0
 1.2
@@
 Wire Wire Line
 	10150 4100 10600 4100
+Text Notes 9750 2850 0    50   ~ 0
+1.5k
 $EndSCHEMATC

Commit message: v1.3 release
Parts:
- added D2: LTST-C191KGKT, leds:LEDC1608X60, symbol Device:LED
- added R2: 470, passive:R_0402_1005Metric_Rounded, symbol Device:R
- TP1, TP2, TP3, TP4: symbol Connector_Specialized:Test_Point -> Connector:TestPoint
- U2: symbol Regulator_Linear:MIC5205-3.3 -> Regulator_Linear:MIC5205-3.3YM5
- U3: symbol MCU_ST_STM32:STM32F103CBUx -> MCU_ST_STM32F1:STM32F103CBUx
Connections:
- wire segments 92 -> 96
Other:
- note added: "1.3"
- note added: "2018-11-18"
- note removed: "1.2"
- note removed: "2018-04-03"
