File: ubmp_v1.sch (KiCad schematic (older format))
At the start: 33 parts, among them J1 Conn_02x05_Counter_Clockwise, J2 USB_A, U1 STM32F103CBUx, U2 MIC5245-3.3, Y1 PRQC8.00CR1010V00L

Commit message: Bumped schematic date
Other:
- note added: "2018-03-27"
- note removed: "2018-02-16"
Changed lines of the file:
@@
 µBMP
 Text Notes 8150 7650 0    67   ~ 0
-2018-02-16
+2018-03-27
 Text Notes 10600 7650 0    67   ~ 0
 1.1

Commit message: Split into hierarchical sheep
Parts:
- removed C1, C2, C3, C4, C7: 100n, ubmp:C_0402_1005Metric_Rounded, symbol Device:C_Small
- removed C5, C6: 4.7u, ubmp:C_0603_1608Metric_Rounded, symbol Device:C_Small
- removed D2: GREEN, ubmp:D_0603_1608Metric_Rounded, symbol Device:LED
- removed F1: MF-FSMF050X-2, ubmp:R_0603_1608Metric_Rounded, symbol Device:Polyfuse_Small
- removed J1: Conn_02x05_Counter_Clockwise, ubmp:2x5_2.54mm_side, symbol Connector_Generic:Conn_02x05_Counter_Clockwise
- removed R10, R11, R12, R13, R3, R4, R5: 100, ubmp:R_0402_1005Metric_Rounded, symbol Device:R
- removed R14, R19, R7, R8: 1.5k, ubmp:R_0402_1005Metric_Rounded, symbol Device:R
- removed R15, R16, R9: 22, ubmp:R_0402_1005Metric_Rounded, symbol Device:R
- removed R2: 470, ubmp:R_0402_1005Metric_Rounded, symbol Device:R
- removed TP1, TP2, TP3, TP4: Test_Point, TestPoint:TestPoint_Pad_D1.0mm, symbol Connector_Specialized:Test_Point
- removed U1: STM32F103CBUx, ubmp:QFN-48-1EP_7x7mm_P0.5mm_EP5.15x5.15mm, symbol MCU_ST_STM32:STM32F103CBUx
- removed U2: MIC5245-3.3, ubmp:SOT-23-5_Rounded, symbol Regulator_Linear:MIC5205-3.3
- removed Y1: PRQC8.00CR1010V00L, ubmp:Resonator_3pin_3.2x1.3mm, symbol Device:Resonator
Connections:
- net labels removed: +3.3V, BMP_RST, BMP_RSTo, BMP_RX, BMP_RXo, BMP_SWCLK_TCK, BMP_SWCLK_TCKo, BMP_SWDIO_TMS, BMP_SWDIO_TMSo, BMP_SWO, BMP_SWOo, BMP_TDI, BMP_TDIo, BMP_TDO, BMP_TDOo, BMP_TX, BMP_TXo, BOOT0, DM_P, DP_P, LED_STLINK, NRST, STM_ID, STM_ID2, SWCLK, SWDIO
- wire segments 98 -> 12
- no-connect marks 21 -> 0
Other:
- note removed: "MCO"
- note removed: "RST resistor is 22 Ohm to support board with small (<1.5k) pullup on RST"
- note removed: "STLink V2 identifier (PC13 = 0)"
- note removed: "SWD Programming"

Commit message: Updated pinput
Changed lines of the file:
@@
 L power:+5V #PWR01
 U 1 1 5A78C20D
-P 10300 4500
-F 0 "#PWR01" H 10300 4350 50  0001 C CNN
-F 1 "+5V" V 10315 4628 50  0000 L CNN
-F 2 "" H 10300 4500 50  0001 C CNN
-F 3 "" H 10300 4500 50  0001 C CNN
-	1    10300 4500
+P 6150 4150
+F 0 "#PWR01" H 6150 4000 50  0001 C CNN
+F 1 "+5V" V 6165 4278 50  0000 L CNN
+F 2 "" H 6150 4150 50  0001 C CNN
+F 3 "" H 6150 4150 50  0001 C CNN
+	1    6150 4150
 	0    -1   -1   0
 $EndComp
@@
 L power:GND #PWR02
 U 1 1 5A78C254
-P 10750 3800
-F 0 "#PWR02" H 10750 3550 50  0001 C CNN
-F 1 "GND" H 10755 3627 50  0000 C CNN
-F 2 "" H 10750 3800 50  0001 C CNN
-F 3 "" H 10750 3800 50  0001 C CNN
-	1    10750 3800
+P 6600 3450
+F 0 "#PWR02" H 6600 3200 50  0001 C CNN
+F 1 "GND" H 6605 3277 50  0000 C CNN
+F 2 "" H 6600 3450 50  0001 C CNN
+F 3 "" H 6600 3450 50  0001 C CNN
+	1    6600 3450
 	-1   0    0    1
 $EndComp
 Wire Wire Line
-	10750 3800 10750 3850
+	6600 3450 6600 3500
 Wire Wire Line
-	10750 3850 10650 3850
+	6600 3500 6500 3500
 Wire Wire Line
-	10650 3850 10650 3900
-Connection ~ 10750 3850
+	6500 3500 6500 3550
+Connection ~ 6600 3500
 Wire Wire Line
-	10750 3850 10750 3900
-Text Label 10200 4300 0    50   ~ 0
+	6600 3500 6600 3550
+Text Label 6050 3950 0    50   ~ 0
 DP
-Text Label 10200 4200 0    50   ~ 0
+Text Label 6050 3850 0    50   ~ 0
 DM
 $Comp
 L Connector_Specialized:USB_A J2
 U 1 1 5A80B5EC
-P 10650 4300
-F 0 "J2" H 10706 4767 50  0000 C CNN
-F 1 "USB_A" H 10706 4676 50  0000 C CNN
-F 2 "usbpcb:USB_A_1001-011-01101" H 10800 4250 50  0001 C CNN
-F 3 "" H 10800 4250 50  0001 C CNN
-	1    10650 4300
+P 6500 3950
+F 0 "J2" H 6556 4417 50  0000 C CNN
+F 1 "USB_A" H 6556 4326 50  0000 C CNN
+F 2 "usbpcb:USB_A_1001-011-01101" H 6650 3900 50  0001 C CNN
+F 3 "" H 6650 3900 50  0001 C CNN
+	1    6500 3950
 	-1   0    0    1
 $EndComp
 Wire Wire Line
-	10300 4500 10350 4500
+	6150 4150 6200 4150
 $Comp
 L power:PWR_FLAG #FLG01
 U 1 1 5A8464BC
-P 10300 4500
-F 0 "#FLG01" H 10300 4575 50  0001 C CNN
-F 1 "PWR_FLAG" H 10300 4674 50  0000 C CNN
-F 2 "" H 10300 4500 50  0001 C CNN
-F 3 "" H 10300 4500 50  0001 C CNN
-	1    10300 4500
+P 6150 4150
+F 0 "#FLG01" H 6150 4225 50  0001 C CNN
+F 1 "PWR_FLAG" H 6150 4324 50  0000 C CNN
+F 2 "" H 6150 4150 50  0001 C CNN
+F 3 "" H 6150 4150 50  0001 C CNN
+	1    6150 4150
 	-1   0    0    1
 $EndComp
-Connection ~ 10300 4500
+Connection ~ 6150 4150
 $Comp
 L power:PWR_FLAG #FLG02
 U 1 1 5A84681F
-P 10650 3850
-F 0 "#FLG02" H 10650 3925 50  0001 C CNN
-F 1 "PWR_FLAG" V 10650 3978 50  0000 L CNN
-F 2 "" H 10650 3850 50  0001 C CNN
-F 3 "" H 10650 3850 50  0001 C CNN
-	1    10650 3850
+P 6500 3500
+F 0 "#FLG02" H 6500 3575 50  0001 C CNN
+F 1 "PWR_FLAG" V 6500 3628 50  0000 L CNN
+F 2 "" H 6500 3500 50  0001 C CNN
+F 3 "" H 6500 3500 50  0001 C CNN
+	1    6500 3500
 	0    -1   -1   0
 $EndComp
-Connection ~ 10650 3850
+Connection ~ 6500 3500
 $Comp
 L Graphic:Logo_Open_Hardware_Small #LOGO1
@@
 Design available at: github.com/korken89/micro-bmp
 $Sheet
-S 8900 4000 700  500
+S 4750 3650 700  500
 U 5ABFD4E7
 F0 "bmp_core" 50
 F1 "bmp_core.sch" 50
-F2 "5V" I R 9600 4400 50
-F3 "DP" I R 9600 4300 50
-F4 "DM" I R 9600 4200 50
-F5 "GND" I R 9600 4100 50
+F2 "5V" I R 5450 4050 50
+F3 "DP" I R 5450 3950 50
+F4 "DM" I R 5450 3850 50
+F5 "GND" I R 5450 3750 50
 $EndSheet
 Wire Wire Line
-	10350 4300 9600 4300
+	6200 3950 5450 3950
 Wire Wire Line
-	9600 4200 10350 4200
+	5450 3850 6200 3850
 Wire Wire Line
-	10650 3900 9750 3900
+	6500 3550 5600 3550
 Wire Wire Line
-	9750 3900 9750 4100
+	5600 3550 5600 3750
 Wire Wire Line
-	9750 4100 9600 4100
-Connection ~ 10650 3900
+	5600 3750 5450 3750
+Connection ~ 6500 3550
 Wire Wire Line
-	10300 4500 10300 4400
+	6150 4150 6150 4050
 Wire Wire Line
-	10300 4400 9600 4400
+	6150 4050 5450 4050
 $EndSCHEMATC

Commit message: Moved libs to external repo
Parts:
- J2: footprint usbpcb:USB_A_1001-011-01101 -> usb:USB_A_1001-011-01101
Changed lines of the file:
@@
 F 0 "J2" H 6556 4417 50  0000 C CNN
 F 1 "USB_A" H 6556 4326 50  0000 C CNN
-F 2 "usbpcb:USB_A_1001-011-01101" H 6650 3900 50  0001 C CNN
+F 2 "usb:USB_A_1001-011-01101" H 6650 3900 50  0001 C CNN
 F 3 "" H 6650 3900 50  0001 C CNN
 	1    6500 3950

Commit message: Fixed through holes on USB connector to be NPTH
Parts:
- J2: value USB_A -> 1001-011-01101
Changed lines of the file:
@@
 EESchema Schematic File Version 4
-LIBS:ubmp_v1-cache
 EELAYER 26 0
 EELAYER END
@@
 U 1 1 5A80B5EC
 P 6500 3950
-F 0 "J2" H 6556 4417 50  0000 C CNN
-F 1 "USB_A" H 6556 4326 50  0000 C CNN
+F 0 "J2" H 6350 4300 50  0000 C CNN
+F 1 "1001-011-01101" V 6250 3950 50  0000 C CNN
 F 2 "usb:USB_A_1001-011-01101" H 6650 3900 50  0001 C CNN
 F 3 "" H 6650 3900 50  0001 C CNN

Commit message: v1.3 release
Parts:
- J2: symbol Connector_Specialized:USB_A -> Connector:USB_A
Other:
- note added: "1.3"
- note added: "2018-11-18"
- note removed: "1.1"
- note removed: "2018-03-27"
Changed lines of the file:
@@
 DM
 $Comp
-L Connector_Specialized:USB_A J2
+L Connector:USB_A J2
 U 1 1 5A80B5EC
 P 6500 3950
@@
 µBMP
 Text Notes 8150 7650 0    67   ~ 0
-2018-03-27
+2018-11-18
 Text Notes 10600 7650 0    67   ~ 0
-1.1
+1.3
 Text Notes 7100 6850 0    79   ~ 0
 Note that this board is designed to work with the \nSTLink V2 version of Black Magic Probe firmware.
@@
 Wire Wire Line
 	5600 3750 5450 3750
-Connection ~ 6500 3550
 Wire Wire Line
 	6150 4150 6150 4050

Commit message: Moved to USB-C plug
Parts:
- removed J2: 1001-011-01101, usb:USB_A_1001-011-01101, symbol Connector:USB_A
- added P1: USB_C_Plug, usb:USB_C_Plug_Molex_1054440001, symbol Connector:USB_C_Plug
- added R3: 5.1k, passive:R_0402_1005Metric_Rounded, symbol Device:R
Connections:
- wire segments 12 -> 16
- no-connect marks 0 -> 11
Changed lines of the file:
@@
 L power:GND #PWR02
 U 1 1 5A78C254
-P 6600 3450
-F 0 "#PWR02" H 6600 3200 50  0001 C CNN
-F 1 "GND" H 6605 3277 50  0000 C CNN
-F 2 "" H 6600 3450 50  0001 C CNN
-F 3 "" H 6600 3450 50  0001 C CNN
-	1    6600 3450
+P 6650 2450
+F 0 "#PWR02" H 6650 2200 50  0001 C CNN
+F 1 "GND" H 6655 2277 50  0000 C CNN
+F 2 "" H 6650 2450 50  0001 C CNN
+F 3 "" H 6650 2450 50  0001 C CNN
+	1    6650 2450
 	-1   0    0    1
 $EndComp
-Wire Wire Line
-	6600 3450 6600 3500
-Wire Wire Line
-	6600 3500 6500 3500
-Wire Wire Line
-	6500 3500 6500 3550
-Connection ~ 6600 3500
-Wire Wire Line
-	6600 3500 6600 3550
 Text Label 6050 3950 0    50   ~ 0
 DP
 Text Label 6050 3850 0    50   ~ 0
 DM
-$Comp
-L Connector:USB_A J2
-U 1 1 5A80B5EC
-P 6500 3950
-F 0 "J2" H 6350 4300 50  0000 C CNN
-F 1 "1001-011-01101" V 6250 3950 50  0000 C CNN
-F 2 "usb:USB_A_1001-011-01101" H 6650 3900 50  0001 C CNN
-F 3 "" H 6650 3900 50  0001 C CNN
-	1    6500 3950
-	-1   0    0    1
-$EndComp
-Wire Wire Line
-	6150 4150 6200 4150
 $Comp
 L power:PWR_FLAG #FLG01
@@
 L power:PWR_FLAG #FLG02
 U 1 1 5A84681F
-P 6500 3500
-F 0 "#FLG02" H 6500 3575 50  0001 C CNN
-F 1 "PWR_FLAG" V 6500 3628 50  0000 L CNN
-F 2 "" H 6500 3500 50  0001 C CNN
-F 3 "" H 6500 3500 50  0001 C CNN
-	1    6500 3500
+P 6650 2450
+F 0 "#FLG02" H 6650 2525 50  0001 C CNN
+F 1 "PWR_FLAG" V 6650 2578 50  0000 L CNN
+F 2 "" H 6650 2450 50  0001 C CNN
+F 3 "" H 6650 2450 50  0001 C CNN
+	1    6650 2450
 	0    -1   -1   0
 $EndComp
-Connection ~ 6500 3500
 $Comp
 L Graphic:Logo_Open_Hardware_Small #LOGO1
@@
 $EndSheet
 Wire Wire Line
-	6200 3950 5450 3950
-Wire Wire Line
-	5450 3850 6200 3850
-Wire Wire Line
-	6500 3550 5600 3550
-Wire Wire Line
-	5600 3550 5600 3750
-Wire Wire Line
-	5600 3750 5450 3750
-Wire Wire Line
 	6150 4150 6150 4050
 Wire Wire Line
 	6150 4050 5450 4050
+$Comp
+L Connector:USB_C_Plug P1
+U 1 1 5C2E3425
+P 8200 4050
+F 0 "P1" H 7770 3748 50  0000 R CNN
+F 1 "USB_C_Plug" H 7770 3839 50  0000 R CNN
+F 2 "usb:USB_C_Plug_Molex_1054440001" H 8350 4050 50  0001 C CNN
+F 3 "https://www.usb.org/sites/default/files/documents/usb_type-c.zip" H 8350 4050 50  0001 C CNN
+	1    8200 4050
+	-1   0    0    1
+$EndComp
+$Comp
+L Device:R R?
+U 1 1 5C2E65F4
+P 7150 4850
+AR Path="/5ABFD4E7/5C2E65F4" Ref="R?"  Part="1"
+AR Path="/5C2E65F4" Ref="R3"  Part="1"
+F 0 "R3" V 7050 4850 50  0000 C CNN
+F 1 "5.1k" V 7150 4850 50  0000 C CNN
+F 2 "passive:R_0402_1005Metric_Rounded" V 7080 4850 50  0001 C CNN
+F 3 "~" H 7150 4850 50  0001 C CNN
+	1    7150 4850
+	0    1    1    0
+$EndComp
+NoConn ~ 7600 2750
+NoConn ~ 7600 2850
+NoConn ~ 7600 3050
+NoConn ~ 7600 3150
+NoConn ~ 7600 3350
+NoConn ~ 7600 3450
+NoConn ~ 7600 3650
+NoConn ~ 7600 3750
+NoConn ~ 7600 3950
+NoConn ~ 7600 4050
+NoConn ~ 7600 4750
+Wire Wire Line
+	7300 4850 7600 4850
+$Comp
+L power:GND #PWR0101
+U 1 1 5C2E6F9E
+P 7000 4850
+F 0 "#PWR0101" H 7000 4600 50  0001 C CNN
+F 1 "GND" H 7005 4677 50  0000 C CNN
+F 2 "" H 7000 4850 50  0001 C CNN
+F 3 "" H 7000 4850 50  0001 C CNN
+	1    7000 4850
+	0    1    1    0
+$EndComp
+Wire Wire Line
+	7600 5050 6400 5050
+Wire Wire Line
+	6400 5050 6400 4150
+Wire Wire Line
+	6150 4150 6400 4150
+Wire Wire Line
+	6650 2450 6650 3750
+Connection ~ 6650 2450
+Wire Wire Line
+	6650 2450 8200 2450
+Wire Wire Line
+	8200 2450 8500 2450
+Connection ~ 8200 2450
+Wire Wire Line
+	7200 3950 7200 4350
+Wire Wire Line
+	7200 4350 7600 4350
+Wire Wire Line
+	5450 3950 7200 3950
+Wire Wire Line
+	7600 4550 7100 4550
+Wire Wire Line
+	7100 4550 7100 3850
+Wire Wire Line
+	5450 3850 7100 3850
+Wire Wire Line
+	5450 3750 6650 3750
 $EndSCHEMATC
